File: PCB/transmitter/transmitter.kicad_sch (KiCad schematic)
At the start: 28 parts, among them J1 Conn_01x20, J2 Conn_01x20, J3 Conn_01x05, Q1 BC546, Q2 BC546, Q3 BC546, Q4 BC546, Q5 BC546, SW1 SW_MEC_5G, SW2 SW_MEC_5G

Commit message: AUDIO PREPROCESSING: adjust frame count.
Parts:
- removed D5: LED_B, symbol Device:LED
- removed Q5: BC546, Package_TO_SOT_THT:TO-92_Inline, symbol Transistor_BJT:BC546
- removed R10: R, symbol Device:R
- removed R9: 1k, symbol Device:R
- removed SW1, SW2: SW_MEC_5G, symbol Switch:SW_MEC_5G
- added C2: 100n, Capacitor_THT:C_Disc_D3.0mm_W1.6mm_P2.50mm, symbol Device:C
- added R13: 10k, Resistor_THT:R_Axial_DIN0207_L6.3mm_D2.5mm_P7.62mm_Horizontal, symbol Device:R
- added R14: 1k, Resistor_THT:R_Axial_DIN0207_L6.3mm_D2.5mm_P7.62mm_Horizontal, symbol Device:R
- added S1, S2: 1825967-1, 1825967-1:SW_1825967-1, symbol 1825967-1:1825967-1
- C1: value C -> 100n; footprint (none) -> Capacitor_THT:C_Disc_D3.0mm_W1.6mm_P2.50mm
- D1: footprint (none) -> LED_THT:LED_D3.0mm
- D2, D3, D4: footprint (none) -> LED_THT:LED_D5.0mm
- J3: footprint (none) -> Connector_PinSocket_2.54mm:PinSocket_1x05_P2.54mm_Vertical
- R1, R4: value R -> 100R; footprint (none) -> Resistor_THT:R_Axial_DIN0207_L6.3mm_D2.5mm_P7.62mm_Horizontal
- R11, R12: value R -> 4k7; footprint (none) -> Resistor_THT:R_Axial_DIN0207_L6.3mm_D2.5mm_P7.62mm_Horizontal
- R2, R3, R5, R7: footprint (none) -> Resistor_THT:R_Axial_DIN0207_L6.3mm_D2.5mm_P7.62mm_Horizontal
- R6: value R -> 80R; footprint (none) -> Resistor_THT:R_Axial_DIN0207_L6.3mm_D2.5mm_P7.62mm_Horizontal
- R8: value R -> 120R; footprint (none) -> Resistor_THT:R_Axial_DIN0207_L6.3mm_D2.5mm_P7.62mm_Horizontal
Connections:
- net ADC_0: now also C1.2, R11.2, R12.1
- net BUTTON: now also J2.1 (Pin_1), C2.1, R14.1; no longer J1.20 (Pin_20)
- net GND: now also J3.1 (Pin_1), C2.2, S1.3, S1.4, S2.3, S2.4; no longer J3.5 (Pin_5)
- net RUN: now also S2.1, S2.2
- net at C1.1: now also J3.4 (Pin_4); no longer J3.2 (Pin_2)
- net 3V3 renamed +3V3
- net +3V3: now also R13.2
- net 5V renamed +5V
- net +5V: now also J3.2 (Pin_2); no longer J3.4 (Pin_4)
- net A3V3: no longer names the net of J2.15 (Pin_15)
- net LED_B: no longer names the net of J1.6 (Pin_6)
- new net: R13.1, R14.2, S1.1, S1.2
- no-connect marks 22 -> 24
Other:
- note added: "GPIO15 BUTTON"
- note added: "RUN BUTTON"
- note removed: "BLUE"
- moved on the sheet: C1, J1, J2, J3, R1, R11, R12, R4, R6, R8
